File: 3. Eagle/wirelessSensor 0.1.brd (EAGLE design)
At the start: 25.1 x 25.4 mm, 15 parts, among them U1 HDC1080, U2 PIC16F1823-X_SL, X1 22-23-2021

Commit message: Started work on the I2C interface, and organized the code a bit more
Parts:
- added R1, R2: 4.7k, rcl:R0603
Connections:
- net N$2: now also R1.1
- net N$3: now also R2.1
- net VCC: now also R1.2, R2.2
Changed lines of the file:
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@@
 <attribute name="MPN" value="22-23-2021" x="21.59" y="21.59" size="1.778" layer="27" rot="R180" display="off"/>
 </element>
+<element name="R1" library="rcl" package="R0603" value="4.7k" x="6.35" y="10.16"/>
+<element name="R2" library="rcl" package="R0603" value="4.7k" x="6.35" y="7.62"/>
 </elements>
 <signals>
@@
 </signal>
 <signal name="VCC">
+<contactref element="C1" pad="1"/>
+<contactref element="X1" pad="1"/>
+<contactref element="ESP8266" pad="8"/>
+<contactref element="R2" pad="2"/>
+<contactref element="R1" pad="2"/>
 <contactref element="U2" pad="1"/>
 <contactref element="U1" pad="5"/>
@@
 <contactref element="U2" pad="3"/>
 <contactref element="C2" pad="1"/>
-<contactref element="C1" pad="1"/>
-<contactref element="X1" pad="1"/>
-<contactref element="ESP8266" pad="8"/>
 <wire x1="19.47" y1="16.51" x2="22.86" y2="21.59" width="0" layer="19" extent="1-1"/>
 <wire x1="17.9578" y1="13.97" x2="19.47" y2="16.51" width="0" layer="19" extent="1-1"/>
@@
 <wire x1="5.209996875" y1="16.51" x2="7.62" y2="17.36" width="0" layer="19" extent="1-1"/>
 <wire x1="3.81" y1="24.13" x2="5.209996875" y2="16.51" width="0" layer="19" extent="1-1"/>
+<wire x1="7.2" y1="10.16" x2="16.51" y2="3.81" width="0" layer="19" extent="1-1"/>
+<wire x1="7.2" y1="7.62" x2="7.2" y2="10.16" width="0" layer="19" extent="1-1"/>
 </signal>
 <signal name="GND">
@@
 <contactref element="U1" pad="6"/>
 <contactref element="SCL" pad="TP"/>
+<contactref element="R1" pad="1"/>
 <wire x1="5.209996875" y1="17.509996875" x2="22.6822" y2="8.89" width="0" layer="19" extent="1-1"/>
 <wire x1="1.27" y1="10.16" x2="5.209996875" y2="17.509996875" width="0" layer="19" extent="1-1"/>
+<wire x1="5.5" y1="10.16" x2="1.27" y2="10.16" width="0" layer="19" extent="1-1"/>
 </signal>
 <signal name="N$3">
@@
 <contactref element="U1" pad="1"/>
 <contactref element="SDA" pad="TP"/>
-<wire x1="2.410003125" y1="17.509996875" x2="22.6822" y2="7.62" width="0" layer="19" extent="1-1"/>
-<wire x1="1.27" y1="7.62" x2="2.410003125" y2="17.509996875" width="0" layer="19" extent="1-1"/>
+<contactref element="R2" pad="1"/>
+<wire x1="1.27" y1="7.62" x2="22.6822" y2="7.62" width="0" layer="19" extent="1-1"/>
+<wire x1="2.410003125" y1="17.509996875" x2="1.27" y2="7.62" width="0" layer="19" extent="1-1"/>
+<wire x1="5.5" y1="7.62" x2="1.27" y2="7.62" width="0" layer="19" extent="1-1"/>
 </signal>
 <signal name="N$4">
